File: electronics/board1/pcb/Attiny85_USB/.kiri/Attiny85_USB.kicad_sch (KiCad schematic)
At the start: 12 parts, among them J1 Conn_01x04, J2 Conn_01x04, U1 ATtiny85-20M

Commit message: Add files via upload
Parts:
- added C2: C, Capacitor_SMD:C_0201_0603Metric, symbol Device:C
- added D8: W01G, Diode_THT:Diode_Bridge_Round_D9.8mm, symbol Diode_Bridge:W01G
- added R5, R6, R7: R, Resistor_SMD:R_0508_1220Metric_Pad1.12x2.15mm_HandSolder, symbol Device:R
- added T1: CST1, Transformer_SMD:Transformer_Coilcraft_CST1, symbol Transformer:CST1
Connections:
- new net: R6.2, T1.6
- new net: C2.2, D8.3 (-), R7.1
- new net: C2.1, D8.1 (+), R7.2
- new net: D8.2, T1.7
- new net: R5.1, T1.8
- new net: D8.4, R5.2
