File: electronics/board1/pcb/board1.kicad_sch (KiCad schematic)
At the start: 2 parts

Commit message: kiri test
Parts:
- added D2: LED, symbol Device:LED
- added R2: 2k, symbol Device:R
Connections:
- net +5V: now also R2.1
- net GND: now also D2.1 (K)
- new net: D2.2 (A), R2.2
